File: pico_driver/pico_driver.kicad_pcb (KiCad board)
At the start: 4 copper layers, 65 x 56 mm, 27 parts, among them J1 GPIO, J4 Conn_01x12_Pin, J5 PICO_5VOUT, SW4_UP SW_Push, SW5_UP SW_Push, U1 CAT24C256, U2 Pico

Commit message: update pcb layout
Parts:
- removed C1: 100n, Capacitor_SMD:C_0805_2012Metric
- removed ESC: Conn_ESC, Connector_PinHeader_2.54mm:PinHeader_1x03_P2.54mm_Vertical
- removed JP1: ID_WP, Jumper:SolderJumper-2_P1.3mm_Bridged_Pad1.0x1.5mm
- removed OFF    ON: SW_SPDT, Button_Switch_THT:SW_E-Switch_EG1271_SPDT
- removed R1, R2: 3.9k, Resistor_SMD:R_1206_3216Metric
- removed SRV: Conn_SERVO, Connector_PinHeader_2.54mm:PinHeader_1x03_P2.54mm_Vertical
- removed SW4_UP, SW5_UP: SW_Push, Button_Switch_THT:SW_PUSH_6mm_H5mm
- removed U2: Pico, Pico:RPi_Pico_SMD_TH
- added J2: SRV, Connector_PinHeader_2.54mm:PinHeader_1x03_P2.54mm_Horizontal, F.Cu at (114.3, 95.8)
- added J3: ESC, Connector_PinHeader_2.54mm:PinHeader_1x03_P2.54mm_Vertical, F.Cu at (114.3, 90.8)
- added J6: VBUS_OUT, Connector_PinHeader_2.54mm:PinHeader_1x02_P2.54mm_Vertical, F.Cu at (162.7, 86.4)
- added J7: 3V3_OUT, Connector_PinHeader_2.54mm:PinHeader_1x02_P2.54mm_Vertical, F.Cu at (154.1, 80.9)
- added J8: FUNC, Connector_PinHeader_2.54mm:PinHeader_1x04_P2.54mm_Vertical, F.Cu at (155.4, 68.0)
- added SW1: SW_SPDT, Button_Switch_THT:SW_E-Switch_EG1271_SPDT, F.Cu at (106.3, 72.3)
- added SW2: SW_Push, Button_Switch_THT:SW_PUSH_6mm_H5mm, F.Cu at (129.5, 95.8)
- added SW3: SW_Push, Button_Switch_THT:SW_PUSH_6mm_H5mm, F.Cu at (143.7, 89.2)
- C2, C3: footprint Capacitor_SMD:C_0805_2012Metric -> Capacitor_SMD:C_0805_2012Metric_Pad1.18x1.45mm_HandSolder
- J4: value Conn_01x12_Pin -> ADC; footprint Connector_PinHeader_2.54mm:PinHeader_1x12_P2.54mm_Vertical -> Connector_PinHeader_2.54mm:PinHeader_1x05_P2.54mm_Vertical
- J5: value PICO_5VOUT -> GP_Breakout; footprint Connector_PinHeader_2.54mm:PinHeader_1x02_P2.54mm_Vertical -> Connector_PinHeader_2.54mm:PinHeader_1x10_P2.54mm_Vertical
- U1: value CAT24C256 -> Pico; footprint CAT24C256:TSSOP8_4P50X3P10_ONS -> RaspberryPi_Pico:RaspberryPi_Pico_Common_THT
- moved G*** 40.2 mm to (122.5, 91.1)
- moved J5 32.7 mm to (163.0, 53.3), turned to -90 degrees
- moved J4 30.1 mm to (150.3, 80.9), turned to -90 degrees
- moved U1 26.1 mm to (163.0, 58.5), turned to -90 degrees
- moved D1 14.3 mm to (108.8, 84.3), turned to 90 degrees
- moved C3 4.54 mm to (136.1, 80.4)
- moved R7 4.53 mm to (136.6, 84.0)
- moved R3 4.01 mm to (118.9, 83.0)
- moved R4 4.01 mm to (121.9, 83.0)
- moved R5 4.01 mm to (124.9, 83.0)
- moved C2 3.74 mm to (131.0, 80.4)
- moved R6 3.52 mm to (131.5, 84.0)
Connections:
- J4 pad 1: /GP0 -> /ADC_VREF
- J4 pad 2: /GP1 -> /ADC2
- J4 pad 3: /GP2 -> GND
- J4 pad 4: /GP3 -> /ADC1
- J4 pad 5: /GP4 -> /ADC0
- J5 pad 1: VBUS -> /GP0
- J5 pad 2: GND -> /GP1
- R6 pad 2: +3V3_PICO -> 3V3_OUT
- R7 pad 2: +3V3_PICO -> 3V3_OUT
- U1 pad 1: unconnected-(U1-A0-Pad1) -> /GP0
- U1 pad 2: unconnected-(U1-A1-Pad2) -> /GP1
- U1 pad 3: unconnected-(U1-A2-Pad3) -> GND
- U1 pad 4: GND -> /GP2
- U1 pad 5: /ID_SDA -> /GP3
- U1 pad 6: /ID_SCL -> /GP4
- U1 pad 7: Net-(JP1-A) -> /GP5
- U1 pad 8: +3V3 -> GND
Routing:
- net VSYS: track 57.4 -> 0.00 mm
- net /GP21: track 40.8 -> 0.00 mm
- net +5V: track 38.6 -> 0.00 mm
- net /GP22: track 34.7 -> 0.00 mm
- net +3V3: track 34.5 -> 0.00 mm, vias 1 -> 0
- net /GP7: track 32.2 -> 0.00 mm
- net /GP6: track 28.6 -> 0.00 mm
- net /CE0: track 27.6 -> 0.00 mm
- net +3V3_PICO: track 24.2 -> 0.00 mm
- net /RXD: track 23.3 -> 0.00 mm, vias 1 -> 0
- net /TXD: track 22.6 -> 0.00 mm, vias 1 -> 0
- net /GP5: track 22.5 -> 0.00 mm
- net /GP28: track 21.7 -> 0.00 mm
- net /ADC_VREF: track 19.8 -> 0.00 mm
- net /GP4: track 19.1 -> 0.00 mm
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Other:
- board text added: "BC Cerebellum V2025.04"
- board text removed: "ADC_VREF"
- board text removed: "BC Driver V2025.04"

Commit message: wire up pcb
Parts:
- moved J2 0.35 mm to (114.3, 95.5)
- moved J3 0.35 mm to (114.3, 90.4)
- moved J6 0.33 mm to (163.0, 86.4)
- moved D1 0.26 mm to (108.8, 84.6)
Routing:
- net VSYS: track 0.00 -> 56.9 mm
- net 3V3_OUT: track 0.00 -> 30.3 mm
- net /RXD: track 0.00 -> 25.4 mm
- net /TXD: track 0.00 -> 25.2 mm
- net /SERVO_SIG: track 0.00 -> 22.9 mm
- net +5V: track 0.00 -> 22.0 mm
- net /SW2: track 0.00 -> 21.7 mm, vias 0 -> 2
- net /SW1: track 0.00 -> 21.2 mm
- net /CE0: track 0.00 -> 20.5 mm
- net Net-(D1-BA): track 0.00 -> 18.8 mm
- net /ESC_SIG: track 0.00 -> 16.8 mm
- net /RUN: track 0.00 -> 16.1 mm
- net Net-(D1-GA): track 0.00 -> 14.9 mm
- net /MOSI: track 0.00 -> 12.7 mm
- net /SDA: track 0.00 -> 12.4 mm
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Other:
- board text added: "3V3"
- board text removed: "GP17"
- board text removed: "GP2"
- board text removed: "GP22"
- board text removed: "GP28"
- board text removed: "GP3"
- board text removed: "GP4"
- board text removed: "GP5"
- board text removed: "GP6"
